File: hamboard/stepper_driver.kicad_sch (KiCad schematic)
At the start: 11 parts, among them J8 STEPPER, U5 TMC2130-LA

Commit message: board: bom
Parts:
- added C33: 100nF, Capacitor_SMD:C_0805_2012Metric, symbol Device:C
- added R3: 9k1, Resistor_SMD:R_0805_2012Metric, symbol Device:R
- C15: value 22n -> 22nF
- C17: value 470n -> 470nF
- C19: value 100nF -> 1uF
- C21: value C -> 10nF
- C28: footprint Capacitor_SMD:CP_Elec_8x10 -> Capacitor_SMD:CP_Elec_6.3x7.7; LCSC (none) -> C88677
- J8: footprint Connector_Phoenix_MSTB:PhoenixContact_MSTBA_2,5_4-G-5,08_1x04_P5.08mm_Horizontal -> TerminalBlock:TerminalBlock_bornier-4_P5.08mm; LCSC (none) -> C557656
- U5: LCSC (none) -> C915795
Connections:
- net +24V: now also C33.1
- net GND: now also U5.37 (EP), C33.2
- net 5VOUT: now reaches C18.1, R18.2, U5.25 (5VOUT)
- net 5VOUT: now also R3.1
- net at U5.23 (AIN_IREF): now also R3.2
- no-connect marks 0 -> 5
Other:
- moved on the sheet: C19, C20, C21, C28

Commit message: first pcb layout
Connections:
- net at J8.1 (Pin_1): now also U5.15 (OB2); no longer U5.34 (OA1)
- net at J8.2 (Pin_2): now also U5.13 (OB1); no longer U5.32 (OA2)
- net at J8.3 (Pin_3): now also U5.32 (OA2); no longer U5.13 (OB1)
- net at J8.4 (Pin_4): now also U5.34 (OA1); no longer U5.15 (OB2)
- no-connect marks 5 -> 6
Changed lines of the file:
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@@
   )
   (no_connect (at 146.05 138.43))
+  (no_connect (at 123.19 105.41))
   (no_connect (at 123.19 130.81))
   (no_connect (at 123.19 115.57))
@@
     (pin "2")
   )
-  (symbol (lib_id "Connector:Screw_Terminal_01x04") (at 172.72 80.01 0) (unit 1)
-    (in_bom yes) (on_board yes) (fields_autoplaced)
-    (property "Reference" "J8" (id 0) (at 175.26 80.0099 0)
-      (effects (font (size 1.27 1.27)) (justify left))
-    )
-    (property "Value" "STEPPER" (id 1) (at 175.26 82.5499 0)
-      (effects (font (size 1.27 1.27)) (justify left))
-    )
-    (property "Footprint" "TerminalBlock:TerminalBlock_bornier-4_P5.08mm" (id 2) (at 172.72 80.01 0)
-      (effects (font (size 1.27 1.27)) hide)
-    )
-    (property "Datasheet" "~" (id 3) (at 172.72 80.01 0)
-      (effects (font (size 1.27 1.27)) hide)
-    )
-    (property "LCSC" "C557656" (id 4) (at 172.72 80.01 0)
-      (effects (font (size 1.27 1.27)) hide)
-    )
+  (symbol (lib_id "Connector:Screw_Terminal_01x04") (at 172.72 82.55 0) (mirror x) (unit 1)
+    (in_bom yes) (on_board yes) (fields_autoplaced)
+    (property "Reference" "J8" (id 0) (at 172.72 71.12 0))
+    (property "Value" "STEPPER" (id 1) (at 172.72 73.66 0))
+    (property "Footprint" "TerminalBlock:TerminalBlock_bornier-4_P5.08mm" (id 2) (at 172.72 82.55 0)
+      (effects (font (size 1.27 1.27)) hide)
+    )
+    (property "Datasheet" "~" (id 3) (at 172.72 82.55 0)
+      (effects (font (size 1.27 1.27)) hide)
+    )
+    (property "LCSC" "C557656" (id 4) (at 172.72 82.55 0)
+      (effects (font (size 1.27 1.27)) hide)
+    )
