File: hamboard/weight.kicad_sch (KiCad schematic)
At the start: 15 parts, among them J7 weight, Q4 Q_PNP_BCE, U4 HX711

Commit message: board: bom
Parts:
- removed Q4: Q_PNP_BCE, symbol Device:Q_PNP_BCE
- added Q4: MMBT4403, Package_TO_SOT_SMD:SOT-23, symbol Device:Q_PNP_BEC
- C10, C13, C14: value 10uF -> 1uF
- C11: value 10uF -> 100nF
- C12: value 10uF -> 10nF
- C9: value 0.1uF -> 100nF
- J7: LCSC (none) -> C557656
- R14, R15, R16, R17: value 100R -> 100
- U4: LCSC (none) -> C43656
Connections:
- net +3V3: now also Q4.2 (E)
- net at C14.1, J7.1 (Pin_1), R16.2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: now also Q4.3 (C)
- net at U4.2 (BASE): now also Q4.1 (B)
- no-connect marks 0 -> 1
Changed lines of the file:
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@@
   (junction (at 113.03 76.2) (diameter 0) (color 0 0 0 0)
   )
+  (no_connect (at 173.99 96.52))
   (wire (pts (xy 201.93 83.82) (xy 201.93 87.63))
     (stroke (width 0) (type default) (color 0 0 0 0))
@@
   )
   (symbol (lib_id "Device:C") (at 113.03 80.01 0) (unit 1)
-    (in_bom yes) (on_board yes) (fields_autoplaced)
+    (in_bom yes) (on_board yes)
     (property "Reference" "C9" (id 0) (at 116.84 78.7399 0)
       (effects (font (size 1.27 1.27)) (justify left))
     )
-    (property "Value" "0.1uF" (id 1) (at 116.84 81.2799 0)
+    (property "Value" "100nF" (id 1) (at 115.57 81.28 0)
       (effects (font (size 1.27 1.27)) (justify left))
     )
@@
     (pin "1")
     (pin "2")
+  )
+  (symbol (lib_id "Device:Q_PNP_BEC") (at 207.01 78.74 0) (mirror x) (unit 1)
+    (in_bom yes) (on_board yes) (fields_autoplaced)
+    (property "Reference" "Q4" (id 0) (at 212.09 77.4699 0)
+      (effects (font (size 1.27 1.27)) (justify left))
+    )
+    (property "Value" "MMBT4403" (id 1) (at 212.09 80.0099 0)
+      (effects (font (size 1.27 1.27)) (justify left))
+    )
+    (property "Footprint" "Package_TO_SOT_SMD:SOT-23" (id 2) (at 212.09 81.28 0)
+      (effects (font (size 1.27 1.27)) hide)
+    )
+    (property "Datasheet" "https://datasheet.lcsc.com/lcsc/2205061000_Guangdong-Hottech-MMBT4403_C181124.pdf" (id 3) (at 207.01 78.74 0)
+      (effects (font (size 1.27 1.27)) hide)
+    )
+    (property "LCSC" "C181124" (id 4) (at 207.01 78.74 0)
+      (effects (font (size 1.27 1.27)) hide)
+    )
+    (pin "1")
+    (pin "2")
+    (pin "3")
   )
   (symbol (lib_id "Device:R") (at 127.635 62.23 180) (unit 1)
     (in_bom yes) (on_board yes)
     (property "Reference" "R16" (id 0) (at 127.635 62.23 90))
-    (property "Value" "100R" (id 1) (at 125.095 62.23 90))
+    (property "Value" "100" (id 1) (at 125.095 62.23 90))
     (property "Footprint" "Resistor_SMD:R_0805_2012Metric" (id 2) (at 129.413 62.23 90)
       (effects (font (size 1.27 1.27)) hide)
@@
       (effects (font (size 1.27 1.27)) (justify left))
     )
-    (property "Value" "10uF" (id 1) (at 165.1 119.3799 0)
+    (property "Value" "10nF" (id 1) (at 165.1 119.3799 0)
       (effects (font (size 1.27 1.27)) (justify left))
     )
@@
       (effects (font (size 1.27 1.27)) (justify left))
     )
-    (property "Value" "10uF" (id 1) (at 205.74 92.7099 0)
+    (property "Value" "1uF" (id 1) (at 205.74 92.7099 0)
       (effects (font (size 1.27 1.27)) (justify left))
     )
@@
       (effects (font (size 1.27 1.27)) (justify left))
     )
-    (property "Value" "10uF" (id 1) (at 152.4 119.3799 0)
+    (property "Value" "100nF" (id 1) (at 152.4 119.3799 0)
       (effects (font (size 1.27 1.27)) (justify left))
     )
@@
       (effects (font (size 1.27 1.27)) (justify left))
     )
-    (property "Value" "10uF" (id 1) (at 138.43 119.3799 0)
+    (property "Value" "1uF" (id 1) (at 138.43 119.3799 0)
       (effects (font (size 1.27 1.27)) (justify left))
     )
@@
       (effects (font (size 1.27 1.27)) hide)
     )
-    (property "Value" "GND" (id 1) (at 127.635 83.947 90)
+    (property "Value" "GND" (id 1) (at 129.54 78.74 0)
       (effects (font (size 1.27 1.27)) (justify left))
     )
@@
     )
     (pin "1")
-  )
-  (symbol (lib_id "Device:Q_PNP_BCE") (at 207.01 78.74 0) (mirror x) (unit 1)
-    (in_bom yes) (on_board yes) (fields_autoplaced)
-    (property "Reference" "Q4" (id 0) (at 212.09 77.4699 0)
-      (effects (font (size 1.27 1.27)) (justify left))
-    )
-    (property "Value" "Q_PNP_BCE" (id 1) (at 212.09 80.0099 0)
-      (effects (font (size 1.27 1.27)) (justify left))
-    )
-    (property "Footprint" "" (id 2) (at 212.09 81.28 0)
-      (effects (font (size 1.27 1.27)) hide)
-    )
-    (property "Datasheet" "~" (id 3) (at 207.01 78.74 0)
-      (effects (font (size 1.27 1.27)) hide)
-    )
-    (pin "1")
-    (pin "2")
-    (pin "3")
   )
   (symbol (lib_id "Device:R") (at 104.14 81.28 90) (unit 1)
     (in_bom yes) (on_board yes)
     (property "Reference" "R15" (id 0) (at 104.14 81.28 90))
-    (property "Value" "100R" (id 1) (at 104.14 83.82 90))
+    (property "Value" "100" (id 1) (at 104.14 83.82 90))
     (property "Footprint" "Resistor_SMD:R_0805_2012Metric" (id 2) (at 104.14 83.058 90)
       (effects (font (size 1.27 1.27)) hide)
@@
     (property "MAXIMUM_PACKAGE_HEIGHT" "1.8 mm" (id 8) (at 153.67 86.36 0)
       (effects (font (size 1.27 1.27)) (justify left bottom) hide)
+    )
+    (property "LCSC" "C43656" (id 9) (at 153.67 86.36 0)
+      (effects (font (size 1.27 1.27)) hide)
     )
     (pin "1")
@@
     (in_bom yes) (on_board yes)
     (property "Reference" "R17" (id 0) (at 127.635 73.025 90))
-    (property "Value" "100R" (id 1) (at 125.095 73.025 90))
+    (property "Value" "100" (id 1) (at 125.095 73.025 90))
     (property "Footprint" "Resistor_SMD:R_0805_2012Metric" (id 2) (at 129.413 73.025 90)
       (effects (font (size 1.27 1.27)) hide)
@@
   (symbol (lib_id "Device:C") (at 229.235 79.375 0) (unit 1)
     (in_bom yes) (on_board yes) (fields_autoplaced)
-    (property "Reference" "C14" (id 0) (at 233.045 78.1049 0)
-      (effects (font (size 1.27 1.27)) (justify left))
-    )
-    (property "Value" "10uF" (id 1) (at 233.045 80.6449 0)
+    (property "Reference" "C14" (id 0) (at 232.41 78.1049 0)
+      (effects (font (size 1.27 1.27)) (justify left))
+    )
+    (property "Value" "1uF" (id 1) (at 232.41 80.6449 0)
       (effects (font (size 1.27 1.27)) (justify left))
     )
@@
     (in_bom yes) (on_board yes)
     (property "Reference" "R14" (id 0) (at 104.14 78.74 90))
-    (property "Value" "100R" (id 1) (at 104.14 76.2 90))
+    (property "Value" "100" (id 1) (at 104.14 76.2 90))
     (property "Footprint" "Resistor_SMD:R_0805_2012Metric" (id 2) (at 104.14 80.518 90)
       (effects (font (size 1.27 1.27)) hide)
@@
       (effects (font (size 1.27 1.27)) hide)
     )
+    (property "LCSC" "C557656" (id 4) (at 83.82 76.2 0)
+      (effects (font (size 1.27 1.27)) hide)
+    )

Commit message: first pcb layout
Parts:
- J7: footprint Connector_Phoenix_MSTB:PhoenixContact_MSTBA_2,5_4-G-5,08_1x04_P5.08mm_Horizontal -> TerminalBlock:TerminalBlock_bornier-4_P5.08mm
- U4: footprint lib:SOP127P600X180-16N -> SOP127P600X180-16N; symbol HX711:HX711 -> hamboard:HX711
Changed lines of the file:
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@@
     (pin "1")
   )
-  (symbol (lib_id "HX711:HX711") (at 153.67 86.36 0) (unit 1)
+  (symbol (lib_id "hamboard:HX711") (at 153.67 86.36 0) (unit 1)
     (in_bom yes) (on_board yes) (fields_autoplaced)
     (property "Reference" "U4" (id 0) (at 153.67 60.8584 0))
     (property "Value" "HX711" (id 1) (at 153.67 63.3984 0))
-    (property "Footprint" "lib:SOP127P600X180-16N" (id 2) (at 153.67 86.36 0)
+    (property "Footprint" "SOP127P600X180-16N" (id 2) (at 153.67 86.36 0)
       (effects (font (size 1.27 1.27)) (justify left bottom) hide)
     )
@@
       (effects (font (size 1.27 1.27)) (justify left))
     )
-    (property "Footprint" "Connector_Phoenix_MSTB:PhoenixContact_MSTBA_2,5_4-G-5,08_1x04_P5.08mm_Horizontal" (id 2) (at 83.82 76.2 0)
+    (property "Footprint" "TerminalBlock:TerminalBlock_bornier-4_P5.08mm" (id 2) (at 83.82 76.2 0)
       (effects (font (size 1.27 1.27)) hide)
     )

Commit message: board: correct DRC issues
Parts:
- removed TP5: TestPoint, TestPoint:TestPoint_Pad_D1.5mm, symbol Connector:TestPoint
Changed lines of the file:
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@@
     (title "Weight")
-  )
-  (junction (at 182.88 88.9) (diameter 0) (color 0 0 0 0)
   )
   (junction (at 181.61 71.12) (diameter 0) (color 0 0 0 0)
@@
     (stroke (width 0) (type default) (color 0 0 0 0))
   )
-  (wire (pts (xy 182.88 88.9) (xy 186.69 88.9))
+  (wire (pts (xy 173.99 88.9) (xy 186.69 88.9))
     (stroke (width 0) (type default) (color 0 0 0 0))
   )
@@
     (stroke (width 0) (type default) (color 0 0 0 0))
   )
-  (wire (pts (xy 182.88 88.9) (xy 182.88 95.25))
-    (stroke (width 0) (type default) (color 0 0 0 0))
-  )
   (wire (pts (xy 173.99 99.06) (xy 176.53 99.06))
     (stroke (width 0) (type default) (color 0 0 0 0))
@@
   )
   (wire (pts (xy 132.08 96.52) (xy 132.08 100.33))
-    (stroke (width 0) (type default) (color 0 0 0 0))
-  )
-  (wire (pts (xy 173.99 88.9) (xy 182.88 88.9))
     (stroke (width 0) (type default) (color 0 0 0 0))
   )
@@
       (effects (font (size 1.27 1.27)) hide)
     )
-    (pin "1")
-  )
-  (symbol (lib_id "Connector:TestPoint") (at 182.88 95.25 180) (unit 1)
-    (in_bom yes) (on_board yes) (fields_autoplaced)
-    (property "Reference" "TP5" (id 0) (at 185.42 97.2819 0)
-      (effects (font (size 1.27 1.27)) (justify right))
-    )
-    (property "Value" "TestPoint" (id 1) (at 185.42 99.8219 0)
-      (effects (font (size 1.27 1.27)) (justify right))
-    )
-    (property "Footprint" "TestPoint:TestPoint_Pad_D1.5mm" (id 2) (at 177.8 95.25 0)
-      (effects (font (size 1.27 1.27)) hide)
-    )
-    (property "Datasheet" "~" (id 3) (at 177.8 95.25 0)
-      (effects (font (size 1.27 1.27)) hide)
-    )

Commit message: board: fixed esp heat pads
Parts:
- TP4: value TestPoint -> W_CLK
Changed lines of the file:
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@@
       (effects (font (size 1.27 1.27)) hide)
     )
-    (property "Datasheet" "https://datasheet.lcsc.com/lcsc/2205061000_Guangdong-Hottech-MMBT4403_C181124.pdf" (id 3) (at 207.01 78.74 0)
+    (property "Datasheet" "~" (id 3) (at 207.01 78.74 0)
       (effects (font (size 1.27 1.27)) hide)
     )
@@
   )
   (symbol (lib_id "Connector:TestPoint") (at 132.08 100.33 180) (unit 1)
-    (in_bom yes) (on_board yes) (fields_autoplaced)
+    (in_bom yes) (on_board yes)
     (property "Reference" "TP4" (id 0) (at 134.62 102.3619 0)
+      (effects (font (size 1.27 1.27)) (justify right) hide)
+    )
+    (property "Value" "W_CLK" (id 1) (at 129.54 106.045 0)
       (effects (font (size 1.27 1.27)) (justify right))
     )
-    (property "Value" "TestPoint" (id 1) (at 134.62 104.9019 0)
-      (effects (font (size 1.27 1.27)) (justify right))
-    )
