File: hamboard/hamboard.kicad_pcb (KiCad board)
At the start: 2 copper layers, 89.7 x 63 mm, 92 parts, among them J1 i2c, J10 Conn_01x03_Male, J2 Conn_01x24_Male, J3 USB_B_Micro, J4 Screw_Terminal_Btn, J5 Screw_Terminal_01x02, J6 programmer, J7 weight, J8 STEPPER, J9 Barrel_Jack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

Commit message: pcb: Centered
Parts:
- moved C30 87.0 mm to (132.9, 74.8)
- moved Q2 87.0 mm to (131.2, 120.5)
- moved Q3 87.0 mm to (131.2, 116.7)
- moved C10 87.0 mm to (181.5, 78.5)
- moved C11 87.0 mm to (181.5, 80.5)
- moved C12 87.0 mm to (181.5, 82.5)
- moved C16 87.0 mm to (113.3, 114.0)
- moved C17 87.0 mm to (112.0, 110.7)
- moved C18 87.0 mm to (112.0, 106.6)
- moved C2 87.0 mm to (171.8, 116.0)
- moved C26 87.0 mm to (130.8, 100.9)
- moved C31 87.0 mm to (149.8, 67.9)
- moved C6 87.0 mm to (126.4, 123.3)
- moved C8 87.0 mm to (133.4, 123.3)
- moved D1 87.0 mm to (113.7, 119.3)
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